File: Aviator_Controller/Aviator_Controller.kicad_sch (KiCad schematic)
At the start: 9 parts, among them J1 Conn_01x02, J2 Conn_01x04, J3 Conn_01x03, J4 USB_C_Receptacle_USB2.0_16P, Q1 NMOS, U1 STM32F072C8Ux, Y1 Crystal_GND24

Commit message: added the pcb project v0.1
Parts:
- removed C1: C_Small, symbol Device:C_Small
- removed Q1: NMOS, symbol Simulation_SPICE:NMOS
- added C10, C2, C3: 1u, Capacitor_SMD:C_0603_1608Metric_Pad1.08x0.95mm_HandSolder, symbol Device:C_Small
- added C11, C12, C13, C9: 100n, Capacitor_SMD:C_0603_1608Metric_Pad1.08x0.95mm_HandSolder, symbol Device:C_Small
- added C14, C15: 4p, Capacitor_SMD:C_0603_1608Metric_Pad1.08x0.95mm_HandSolder, symbol Device:C_Small
- added C4, C7, C8: 4.7u, Capacitor_SMD:C_0805_2012Metric_Pad1.18x1.45mm_HandSolder, symbol Device:C_Small
- added C5, C6: 10u, Capacitor_SMD:C_0805_2012Metric_Pad1.18x1.45mm_HandSolder, symbol Device:C_Small
- added J10, J11, J12, J13, J14, J15, J16, J17, J18, J19, J20, J21, J9: Conn_01x02, Connector_PinHeader_2.54mm:PinHeader_1x02_P2.54mm_Vertical, symbol Connector_Generic:Conn_01x02
- added J5: Conn_02x03_Counter_Clockwise, Connector_PinHeader_2.54mm:PinHeader_2x03_P2.54mm_Vertical, symbol Connector_Generic:Conn_02x03_Counter_Clockwise
- added J6, J7, J8: Conn_01x03, Connector_PinHeader_2.54mm:PinHeader_1x03_P2.54mm_Vertical, symbol Connector_Generic:Conn_01x03
- added L1: 3.3u, Inductor_SMD:L_Bourns-SRN6028, symbol Device:L
- added Q1, Q2: Q_NMOS_GSD, Package_TO_SOT_SMD:SOT-23, symbol Device:Q_NMOS_GSD
- added R10, R11, R12, R13, R14, R15, R16, R17, R7, R8, R9: 10k, Resistor_SMD:R_0603_1608Metric_Pad0.98x0.95mm_HandSolder, symbol Device:R_Small
- added R18, R19, R20, R21: 1.5k, Resistor_SMD:R_0603_1608Metric_Pad0.98x0.95mm_HandSolder, symbol Device:R_Small
- added R2, R5: 0, Resistor_SMD:R_0603_1608Metric_Pad0.98x0.95mm_HandSolder, symbol Device:R_Small
- added R3, R4: 5.1k, Resistor_SMD:R_0603_1608Metric_Pad0.98x0.95mm_HandSolder, symbol Device:R_Small
- added R6: DNP, Resistor_SMD:R_0603_1608Metric_Pad0.98x0.95mm_HandSolder, symbol Device:R_Small
- added U2: ST1S06PU33R, footprints:DFN_6PU33R_STM, symbol 2024-12-23_11-54-02:ST1S06PU33R
- J1: footprint (none) -> Connector_PinHeader_2.54mm:PinHeader_1x02_P2.54mm_Vertical
- J2: footprint (none) -> Connector_PinHeader_2.54mm:PinHeader_1x04_P2.54mm_Vertical
- J3: footprint (none) -> Connector_PinHeader_2.54mm:PinHeader_1x03_P2.54mm_Vertical
- J4: footprint (none) -> USB4105GFA120:GCT_USB4105GFA120
- R1: value R_Small -> 10k; footprint (none) -> Resistor_SMD:R_0603_1608Metric_Pad0.98x0.95mm_HandSolder
- Y1: value Crystal_GND24 -> ABMM2-8; footprint (none) -> ABMM2-8.000MHZ-E2-T:XTAL_ABMM2-8.000MHZ-E2-T
Connections:
- net Button11: now reaches J1.1 (Pin_1)
- net Button11: now also U1.25 (PB12)
- net GND: now reaches J1.2 (Pin_2)
- net GND: now also J2.1 (Pin_1), J3.2 (Pin_2), J4.A1 (GND), J4.A12 (GND), J4.B1 (GND), J4.B12 (GND), U1.23 (VSS), U1.35 (VSS), U1.47 (VSS), U1.49 (VSS), U1.8 (VSSA), Y1.2, Y1.4, C10.2, C11.2, C12.2, C13.2, C14.1, C15.2, C2.2, C3.2, C4.2, C5.2, C6.2, C7.2, C8.2, C9.2, J10.2 (Pin_2), J11.2 (Pin_2), J12.2 (Pin_2), J13.2 (Pin_2), J14.2 (Pin_2), J15.2 (Pin_2), J16.2 (Pin_2), J17.2 (Pin_2), J18.2 (Pin_2), J19.2 (Pin_2), J5.4 (Pin_4), J6.2 (Pin_2), J7.2 (Pin_2), J8.2 (Pin_2), J9.2 (Pin_2), Q1.2 (S), Q2.2 (S), R15.1, R17.1, R2.2, R3.2, R4.2, R6.2, U2.2 (GND), U2.7 (GND)
- net +3.3V: now reaches U1.1 (VBAT)
- net +3.3V: now also J2.2 (Pin_2), R1.1, U1.24 (VDD), U1.36 (VDDIO2), U1.48 (VDD), U1.9 (VDDA), C10.1, C11.1, C12.1, C13.1, C5.1, C6.1, C7.1, C8.1, C9.1, J5.3 (Pin_3), L1.2, R10.1, R11.1, R12.1, R13.1, R14.1, R18.1, R19.1, R20.1, R21.1, R5.2, R8.1, R9.1
- net EncB1: now reaches U1.10 (PA0)
- net EncB1: now also J3.1 (Pin_1), R1.2
- net EncA1: now reaches U1.11 (PA1)
- net EncA1: now also J3.3 (Pin_3), R8.2
- net Button3: now reaches U1.13 (PA3)
- net Button3: now also J19.1 (Pin_1)
- net Button4: now reaches U1.14 (PA4)
- net Button4: now also J12.1 (Pin_1)
- net Button5: now reaches U1.15 (PA5)
- net Button5: now also J10.1 (Pin_1)
- net EncB2: now reaches U1.16 (PA6)
- net EncB2: now also J6.1 (Pin_1), R10.2
- net EncA2: now reaches U1.17 (PA7)
- net EncA2: now also J6.3 (Pin_3), R9.2
- net Button6: now reaches U1.18 (PB0)
- net Button6: now also J13.1 (Pin_1)
- net Button7: now reaches U1.19 (PB1)
- net Button7: now also J11.1 (Pin_1)
- net Button0: now reaches U1.2 (PC13)
- net Button0: now also J16.1 (Pin_1)
- net Button8: now reaches U1.20 (PB2)
- net Button8: now also J14.1 (Pin_1)
- net Button9: now reaches U1.21 (PB10)
- net Button9: now also J9.1 (Pin_1)
- net Button10: now reaches U1.22 (PB11)
- net Button10: now also J15.1 (Pin_1)
- net EncB3: now reaches U1.27 (PB14)
- net EncB3: now also J7.1 (Pin_1), R12.2
- net EncA3: now reaches U1.28 (PB15)
- net EncA3: now also J7.3 (Pin_3), R11.2
- net EncB0: now reaches U1.29 (PA8)
- net EncB0: now also J8.1 (Pin_1), R14.2
- net Button1: now reaches U1.3 (PC14)
- net Button1: now also J18.1 (Pin_1)
- net EncA0: now reaches U1.30 (PA9)
- net EncA0: now also J8.3 (Pin_3), R13.2
- net D-: now reaches U1.32 (PA11)
- net D-: now also J4.A7 (D-), J4.B7 (D-), R18.2
- net D+: now reaches U1.33 (PA12)
- net D+: now also J4.A6 (D+), J4.B6 (D+), R19.2
- net SWDIO: now reaches U1.34 (PA13)
- net SWDIO: now also J5.6 (Pin_6)
- net SWCLK: now reaches U1.37 (PA14)
- net SWCLK: now also J5.5 (Pin_5)
- net Button2: now reaches U1.4 (PC15)
- net Button2: now also J17.1 (Pin_1)
- net SCL: now reaches U1.42 (PB6)
- net SCL: now also J2.4 (Pin_4), R21.2
- net SDA: now reaches U1.43 (PB7)
- net SDA: now also J2.3 (Pin_3), R20.2
- net BOOT0: now reaches U1.44 (BOOT0)
- net BOOT0: now also J5.2 (Pin_2)
- net out1: now reaches U1.45 (PB8)
- net out1: now also R16.1
- net out2: now reaches U1.46 (PB9)
- net out2: now also R7.1
- net at U1.5 (PF0): now also Y1.3, C14.2
- net at U1.6 (PF1): now also Y1.1, C15.1
- net NRST: now reaches U1.7 (NRST)
- net NRST: now also J5.1 (Pin_1)
- net +5V: now reaches J4.A4 (VBUS), J4.A9 (VBUS), J4.B4 (VBUS), J4.B9 (VBUS)
- net +5V: now also C2.1, C3.1, C4.1, J20.1 (Pin_1), J21.1 (Pin_1), U2.4 (VIN_SW), U2.5 (VIN_A), U2.6 (VINH)
- net at J4.A5 (CC1): now also R4.1
- net at J4.B5 (CC2): now also R3.1
- net at J4.S1 (SHIELD): now also R2.1
- new net: R5.1, R6.1, U2.1 (FB/VO)
- new net: L1.1, U2.3 (SW)
- new net: Q1.1 (G), R15.2, R7.2
- new net: J20.2 (Pin_2), Q1.3 (D)
- new net: Q2.1 (G), R16.2, R17.2
- new net: J21.2 (Pin_2), Q2.3 (D)
- no-connect marks 0 -> 9
Other:
- company: (none) -> AGH KNE
- title: (none) -> AVIATOR HID CONTROLLER
- moved on the sheet: J1, J3, R1, U1, Y1
